File: PowerModule.kicad_pcb (KiCad board)
At the start: 2 copper layers, 38 x 50 mm, 28 parts, among them CON1 Power In, P1 Power Out, P2 Power Out, SW1 Power, U1 LT1617, U2 LD1117DT33

Commit message: Clean
Routing:
- net +5V: track 122.7 -> 105.3 mm
- net -5V: track 58.9 -> 52.4 mm
- net +3.3V: track 67.2 -> 70.3 mm
- net Net-(C4-Pad2): track 19.2 -> 22.0 mm
- net GND: track 22.6 -> 22.5 mm, vias 10 -> 11

Commit message: OSH Park build works
Parts:
- CON1: footprint Connect:JACK_ALIM -> AB1lib:JACK_ALIM
- moved CON1 0.11 mm to (155.1, 111.0)

Commit message: Clean for posting.
Parts:
- CON1: footprint AB1lib:JACK_ALIM -> AB1lib:DC_PWR_JACK
- moved CON1 0.46 mm to (154.7, 110.7)
- moved P1 0.18 mm to (183.9, 117.9)
Changed lines of the file:
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@@
   (net 7 +3.3V)
   (net 8 "Net-(CON1-Pad1)")
-  (net 9 "Net-(CON1-Pad3)")
-  (net 10 "Net-(D1-Pad1)")
-  (net 11 "Net-(D2-Pad1)")
-  (net 12 "Net-(D3-Pad2)")
+  (net 9 "Net-(D1-Pad1)")
+  (net 10 "Net-(D2-Pad1)")
+  (net 11 "Net-(D3-Pad2)")
+  (net 12 "Net-(CON1-Pad3)")
   (net_class Default "This is the default net class."
     (clearance 0.254)
@@
     (fp_line (start -0.5 0.85) (end 0.5 0.85) (layer F.SilkS) (width 0.15))
     (pad 1 smd rect (at -1.25 0 180) (size 1.5 1.25) (layers F.Cu F.Paste F.Mask)
-      (net 10 "Net-(D1-Pad1)"))
+      (net 9 "Net-(D1-Pad1)"))
     (pad 2 smd rect (at 1.25 0 180) (size 1.5 1.25) (layers F.Cu F.Paste F.Mask)
       (net 2 GND))
@@
     (fp_line (start -0.5 0.85) (end 0.5 0.85) (layer F.SilkS) (width 0.15))
     (pad 1 smd rect (at -1.25 0 180) (size 1.5 1.25) (layers F.Cu F.Paste F.Mask)
-      (net 11 "Net-(D2-Pad1)"))
+      (net 10 "Net-(D2-Pad1)"))
     (pad 2 smd rect (at 1.25 0 180) (size 1.5 1.25) (layers F.Cu F.Paste F.Mask)
       (net 2 GND))
@@
       (net 2 GND))
     (pad 2 smd rect (at 1.25 0) (size 1.5 1.25) (layers F.Cu F.Paste F.Mask)
-      (net 12 "Net-(D3-Pad2)"))
+      (net 11 "Net-(D3-Pad2)"))
     (model Capacitors_SMD.3dshapes/C_0805_HandSoldering.wrl
       (at (xyz 0 0 0))
@@
       (net 1 +5V))
     (pad 2 smd rect (at 1.35 0 180) (size 1.5 1.3) (layers F.Cu F.Paste F.Mask)
-      (net 10 "Net-(D1-Pad1)"))
+      (net 9 "Net-(D1-Pad1)"))
     (model Resistors_SMD.3dshapes/R_0805_HandSoldering.wrl
       (at (xyz 0 0 0))
@@
       (net 7 +3.3V))
     (pad 2 smd rect (at 1.35 0 180) (size 1.5 1.3) (layers F.Cu F.Paste F.Mask)
-      (net 11 "Net-(D2-Pad1)"))
+      (net 10 "Net-(D2-Pad1)"))
     (model Resistors_SMD.3dshapes/R_0805_HandSoldering.wrl
       (at (xyz 0 0 0))
@@
       (net 5 -5V))
     (pad 2 smd rect (at 1.35 0 180) (size 1.5 1.3) (layers F.Cu F.Paste F.Mask)
-      (net 12 "Net-(D3-Pad2)"))
+      (net 11 "Net-(D3-Pad2)"))
     (model Resistors_SMD.3dshapes/R_0805_HandSoldering.wrl
       (at (xyz 0 0 0))
@@
   )
   (module AB1lib:4pinTerminal (layer F.Cu)
-    (at 184 118 270)
+    (at 183.896 117.856 270)
     (fp_text reference P1 (at -0.1 5.2 270) (layer F.SilkS)
       (effects (font (size 1.5 1.5) (thickness 0.15)))
@@
     (fp_line (start -10 -3) (end 10 -3) (layer F.SilkS) (width 0.15))
     (fp_line (start -10 4) (end 10 4) (layer F.SilkS) (width 0.15))
-    (pad 3 thru_hole circle (at 2.5 0 270) (size 2.54 2.54) (drill 0.999998) (layers *.Cu *.Mask F.SilkS)
-      (net 2 GND))
-    (pad 2 thru_hole circle (at -2.5 0 270) (size 2.54 2.54) (drill 0.999998) (layers *.Cu *.Mask F.SilkS)
+    (pad 3 thru_hole circle (at 2.5 0 270) (size 2.54 2.54) (drill 1.3) (layers *.Cu *.Mask F.SilkS)
+      (net 2 GND))
+    (pad 2 thru_hole circle (at -2.5 0 270) (size 2.54 2.54) (drill 1.3) (layers *.Cu *.Mask F.SilkS)
       (net 7 +3.3V))
-    (pad 1 thru_hole circle (at -7.5 0 270) (size 2.54 2.54) (drill 0.999998) (layers *.Cu *.Mask F.SilkS)
-      (net 1 +5V))
-    (pad 4 thru_hole circle (at 7.5 0 270) (size 2.54 2.54) (drill 0.999998) (layers *.Cu *.Mask F.SilkS)
+    (pad 1 thru_hole circle (at -7.5 0 270) (size 2.54 2.54) (drill 1.3) (layers *.Cu *.Mask F.SilkS)
+      (net 1 +5V))
+    (pad 4 thru_hole circle (at 7.5 0 270) (size 2.54 2.54) (drill 1.3) (layers *.Cu *.Mask F.SilkS)
       (net 5 -5V))
   )
-  (module AB1lib:JACK_ALIM (layer F.Cu)
-    (at 155.1 110.95)
+  (module AB1lib:DC_PWR_JACK (layer F.Cu)
+    (at 154.686 110.744)
     (descr "module 1 pin (ou trou mecanique de percage)")
     (tags "CONN JACK")
@@
     (fp_line (start -4.1 4.318) (end 5.588 4.318) (layer F.SilkS) (width 0.15))
     (fp_line (start -4.1 -4.318) (end 5.588 -4.318) (layer F.SilkS) (width 0.15))
-    (pad 2 thru_hole circle (at 0 0) (size 4.8006 4.8006) (drill oval 1.016 2.54) (layers *.Cu *.Mask F.SilkS)
-      (net 2 GND))
-    (pad 1 thru_hole rect (at 6.096 0) (size 4.8006 4.8006) (drill oval 1.016 2.54) (layers *.Cu *.Mask F.SilkS)
+    (pad 2 thru_hole circle (at 0 0) (size 4.8 4.8) (drill 3.2) (layers *.Cu *.Mask F.SilkS)
+      (net 2 GND))
+    (pad 1 thru_hole circle (at 6 0) (size 4.8 4.8) (drill 3.2) (layers *.Cu *.Mask F.SilkS)
       (net 8 "Net-(CON1-Pad1)"))
-    (pad 3 thru_hole circle (at 2.286 5.08) (size 4.8006 4.8006) (drill oval 2.54 1.016) (layers *.Cu *.Mask F.SilkS)
-      (net 9 "Net-(CON1-Pad3)"))
+    (pad 3 thru_hole circle (at 3 4.7) (size 4.8 4.8) (drill 3.2) (layers *.Cu *.Mask F.SilkS)
+      (net 12 "Net-(CON1-Pad3)"))
     (model Connect.3dshapes/JACK_ALIM.wrl
       (at (xyz 0 0 0))
@@
   (segment (start 158.55 119.25) (end 161.1 116.7) (width 0.254) (layer F.Cu) (net 8))
   (segment (start 161.1 116.7) (end 161.096 111) (width 0.254) (layer F.Cu) (net 8))
-  (segment (start 160.15 141) (end 156.75 141) (width 0.254) (layer F.Cu) (net 10))
-  (segment (start 160.15 137) (end 156.75 137) (width 0.254) (layer F.Cu) (net 11))
-  (segment (start 160.15 133) (end 156.75 133) (width 0.254) (layer F.Cu) (net 12))
+  (segment (start 160.15 141) (end 156.75 141) (width 0.254) (layer F.Cu) (net 9))
+  (segment (start 160.15 137) (end 156.75 137) (width 0.254) (layer F.Cu) (net 10))
+  (segment (start 160.15 133) (end 156.75 133) (width 0.254) (layer F.Cu) (net 11))
   (zone (net 2) (net_name GND) (layer B.Cu) (hatch edge 0.508)
     (connect_pads (clearance 0.1524))
