File: PowerModule.sch (KiCad schematic (older format))
At the start: 24 parts, among them CON1 Power In, P1 Power Out, P2 Power Out, SW1 Power, U1 LT1617, U2 LD1117DT33

Commit message: OSH Park build works
Parts:
- CON1: footprint Connect:JACK_ALIM -> AB1lib:JACK_ALIM
Other:
- moved on the sheet: C1, C2, C3, C4, C5, C6, C7, CON1, D1, D2, D3, D4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

Commit message: Clean for posting.
Parts:
- CON1: footprint AB1lib:JACK_ALIM -> AB1lib:DC_PWR_JACK
Changed lines of the file:
@@
 F 0 "CON1" H 2050 3300 60  0000 C CNN
 F 1 "Power In" H 2050 2850 60  0000 C CNN
-F 2 "AB1lib:JACK_ALIM" H 2050 3050 60  0001 C CNN
+F 2 "AB1lib:DC_PWR_JACK" H 2050 3050 60  0001 C CNN
 F 3 "" H 2050 3050 60  0000 C CNN
 	1    2050 3050
